File: Board/JoeMBMS2/JoeMBMS_V3.1.kicad_pcb (KiCad board)
At the start: 2 copper layers, 82 x 92 mm, 63 parts, among them J1 5007620481, Q1 BSO615NG, Q2 BSO615NG, Q3 P-Chanel Mosfet, U1 Teensy4.0, U2 SN65HVD230, U3 DCDC 5V, U4 IS281-4, U5 SN65HVD230, U6 DCDC 3.3V, U7 Level Shifter 5V to 3V, U8 Level Shifter 5V to 3V

Commit message: Update Board V3.1
Parts:
- removed R20, R23: 10k, Resistor_SMD:R_0805_2012Metric
- added C10: 100p, Capacitor_SMD:C_0402_1005Metric, F.Cu at (118.6, 60.7)
- added C11: 100p, Capacitor_SMD:C_0402_1005Metric, F.Cu at (114.2, 51.4)
- added C12: 100p, Capacitor_SMD:C_0402_1005Metric, F.Cu at (114.2, 53.3)
- added C13: 100nF, Capacitor_SMD:C_0805_2012Metric, F.Cu at (151.4, 77.4)
- added C14: 100nF, Capacitor_SMD:C_0805_2012Metric, F.Cu at (151.4, 81.7)
- added C9: 100p, Capacitor_SMD:C_0402_1005Metric, F.Cu at (118.6, 62.6)
- added D5: NUP2105L, Package_TO_SOT_SMD:SOT-23, F.Cu at (116.1, 61.6)
- added D6: NUP2105L, Package_TO_SOT_SMD:SOT-23, F.Cu at (111.7, 52.3)
- added D7: D_Zener, Diode_SMD:D_SOD-123, F.Cu at (153.6, 82.2)
- added D8: D_Zener, Diode_SMD:D_SOD-123, F.Cu at (153.7, 76.7)
- added J2: CAN2_T, Connector_PinHeader_2.54mm:PinHeader_1x02_P2.54mm_Vertical, F.Cu at (115.1, 56.4)
- added J3: CAN1_T, Connector_PinHeader_2.54mm:PinHeader_1x02_P2.54mm_Vertical, F.Cu at (119.2, 65.4)
- R19, R22: value 10k -> 20k
- moved C6 79.7 mm to (127.2, 129.5), turned to 180 degrees
- moved U2 52.7 mm to (120.7, 52.3), turned to 180 degrees
- moved C2 51.4 mm to (158.2, 50.8), turned to 90 degrees
- moved U5 49.2 mm to (124.8, 61.3), turned to 180 degrees
- moved R1 48.7 mm to (118.6, 56.1), turned to 180 degrees
- moved C1 46.7 mm to (122.7, 56.1), turned to 0 degrees
- moved R26 44.2 mm to (122.8, 65.1), turned to 180 degrees
- moved C4 43.7 mm to (126.8, 65.1), turned to 0 degrees
- moved R25 38.7 mm to (120.1, 61.8)
- moved R24 29.3 mm to (115.7, 52.7)
- moved U7 24.7 mm to (152.9, 71.2), turned to 0 degrees
- moved U1 24.7 mm to (148.1, 67.0), turned to -90 degrees
- moved 3.3V 22.0 mm to (143.5, 105.2)
- moved U6 21.2 mm to (135.5, 93.9)
- moved R21 18.4 mm to (148.7, 76.5), turned to 180 degrees
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Connections:
- J1 pad A4: J1_CAN2_L -> J1_CAN1_L
- J1 pad B4: J1_CAN2_H -> J1_CAN1_H
- J1 pad C4: J1_CAN2_H -> J1_CAN2_L
- J1 pad D4: J1_CAN2_T2 -> J1_CAN2_H
- J1 pad J3: J1_CAN1_T2 -> unconnected-(J1-PadJ3)
- J1 pad J4: J1_CAN1_L -> unconnected-(J1-PadJ4)
- J1 pad K3: J1_CAN1_H -> unconnected-(J1-PadK3)
- J1 pad K4: J1_CAN1_H -> unconnected-(J1-PadK4)
- R19 pad 1: Net-(R19-Pad1) -> GND
- R22 pad 1: Net-(R22-Pad1) -> GND
- R24 pad 1: J1_CAN2_T2 -> Net-(J2-Pin_2)
- R25 pad 1: J1_CAN1_T2 -> Net-(J3-Pin_2)
Routing:
- net J1_CAN1_H: track 153.6 -> 31.5 mm, vias 1 -> 0
- net J1_CAN1_L: track 147.3 -> 26.1 mm, vias 1 -> 0
- net J1_CAN2_L: track 74.5 -> 40.0 mm
- net Teensy_Serial_TX: track 54.0 -> 85.6 mm
- net Teensy_D-: track 118.4 -> 88.2 mm
- net Teensy_D+: track 118.9 -> 90.6 mm
- net Teensy_CAN1_TX: track 3.24 -> 30.6 mm
- net J1_CAN2_H: track 74.0 -> 47.2 mm, vias 0 -> 1
- net Teensy_IN4: track 8.30 -> 34.6 mm
- net Teensy_CAN1_RX: track 4.15 -> 30.4 mm
- net Teensy_IN3: track 8.30 -> 31.8 mm
- net Teensy_IN1: track 8.30 -> 31.2 mm
- net Teensy_Serial_RX_5V: track 61.3 -> 81.6 mm
- net Teensy_Serial_BMS_RX_5V: track 52.0 -> 31.7 mm
- net Teensy_IN2: track 8.30 -> 27.4 mm
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Other:
- board size 82 x 92 mm -> 68 x 92 mm
