File: Board/JoeMBMS2/JoeMBMS_V3.1.kicad_sch (KiCad schematic)
At the start: 59 parts, among them J1 5007620481, Q1 BSO615NG, Q2 BSO615NG, Q3 P-Chanel Mosfet, U1 Teensy4.0, U2 SN65HVD230, U3 DCDC 5V, U4 IS281-4, U5 SN65HVD230, U6 DCDC 3.3V, U7 Level Shifter 5V to 3V, U8 Level Shifter 5V to 3V

Commit message: Update Board V3.1
Parts:
- removed R20, R23: 10k, Resistor_SMD:R_0805_2012Metric, symbol Device:R
- added C10, C11, C12, C9: 100p, Capacitor_SMD:C_0402_1005Metric, symbol Device:C
- added C13, C14: 100nF, Capacitor_SMD:C_0805_2012Metric, symbol Device:C
- added D5, D6: NUP2105L, Package_TO_SOT_SMD:SOT-23, symbol Power_Protection:NUP2105L
- added D7, D8: D_Zener, Diode_SMD:D_SOD-123, symbol Device:D_Zener
- added J2: CAN2_T, Connector_PinHeader_2.54mm:PinHeader_1x02_P2.54mm_Vertical, symbol Connector:Conn_01x02_Pin
- added J3: CAN1_T, Connector_PinHeader_2.54mm:PinHeader_1x02_P2.54mm_Vertical, symbol Connector:Conn_01x02_Pin
- C5, C8: LCSC C2972719 -> C3001246
- C6, C7: LCSC C127971 -> C3001246
- J1: footprint Molex_5007620481:5007620481 -> Molex_48_Pin:5007620481
- R19, R22: value 10k -> 20k; LCSC C17414 -> C4328
- U4: footprint TLP2934:TLP293-4 -> TLP293-4:TLP293-4
Connections:
- net GND: now also R19.1, R22.1, C10.1, C11.2, C12.1, C13.1, C14.1, C9.1, D5.3 (A), D6.3 (A), D7.2 (A), D8.2 (A)
- net J1_CAN1_H: now also J1.B4, C9.2, D5.2 (K), J3.1 (Pin_1); no longer J1.K3, J1.K4
- net J1_CAN1_L: now also J1.A4, C10.2, D5.1 (K); no longer J1.J4
- net J1_CAN2_H: now also J1.D4, C12.2, D6.2 (K), J2.1 (Pin_1); no longer J1.B4, J1.C4
- net J1_CAN2_L: now also J1.C4, C11.1, D6.1 (K); no longer J1.A4
- net Teensy_ASEN1: now also C13.2, D8.1 (K)
- net Teensy_ASEN2: now also C14.2, D7.1 (K)
- net J1_CAN1_T2: no longer names the net of J1.J3
- net J1_CAN1_T2: no longer R25.1
- net J1_CAN2_T2: no longer names the net of R24.1
- net J1_CAN2_T2: now also J2.2 (Pin_2); no longer J1.D4
- new net: J3.2 (Pin_2), R25.1
- no-connect marks 38 -> 42
Other:
- note added: "12V"
- note added: "12V Outputs"
- note added: "3V"
- note added: "48-Pin Molex Connector"
- note added: "5V"
- note added: "Analogue Sensor Inputs"
- note added: "CAN 1"
- note added: "CAN 2"
- note added: "GND PWM-Outputs"
- note added: "Isolated Inputs"
- note added: "Level-Shifter for Serial Inputs"
- note added: "Microcontroller"
- note added: "Power Supply"
- moved on the sheet: C1, C2, C3, C4, C5, C6, C7, C8, D1, D2, D3, D4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
