File: Board/JoeM_BMC_V3.2/JoeM_BMC_V3.2.kicad_pcb (KiCad board)
At the start: 2 copper layers, 68 x 92 mm, 70 parts, among them J1 5007620481, J2 CAN2_T, J3 CAN1_T, Q1 BSO615NG, Q2 BSO615NG, Q3 P-Chanel Mosfet, U1 Teensy4.0, U2 SN65HVD230, U3 DCDC 5V, U4 IS281-4, U5 SN65HVD230, U6 DCDC 3.3V, U7 Level Shifter 5V to 3V, U8 Level Shifter 5V to 3V

Commit message: no changes
Parts:
- moved C7 1.97 mm to (153.4, 120.4)
Changed lines of the file:
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@@
 	(footprint "Capacitor_SMD:C_Elec_6.3x7.7"
 		(layer "F.Cu")
-		(at 153.392 122.35 -90)
+		(at 153.37 120.3825 -90)
 		(descr "SMD capacitor, aluminum electrolytic nonpolar, 6.3x7.7mm")
 		(tags "capacitor electrolyic nonpolar")
@@
 			(at 0 1.55 0)
 			(layer "F.Fab")
+			(hide yes)
 			(effects
 				(font
@@
 	)
 	(segment
-		(start 153.392 127.6)
-		(end 153.392 124.8875)
+		(start 153.37 125.6325)
+		(end 153.37 122.92)
 		(width 0.8)
 		(layer "F.Cu")
@@
 	)
 	(segment
-		(start 152.884 127.6)
-		(end 153.9 127.6)
+		(start 152.862 125.6325)
+		(end 153.878 125.6325)
 		(width 0.8)
 		(layer "F.Cu")
@@
 	)
 	(via
-		(at 152.884 127.6)
+		(at 152.862 125.6325)
 		(size 0.8)
 		(drill 0.4)
@@
 	)
 	(via
-		(at 153.9 127.6)
+		(at 153.878 125.6325)
 		(size 0.8)
 		(drill 0.4)
@@
 		(polygon
 			(pts
-				(xy 108.585 56.769) (xy 117.348 68.064) (xy 129.7 68.1) (xy 135.9 74.3) (xy 135.884 122.4) (xy 162.264 122.4)
+				(xy 108.585 56.769) (xy 117.348 68.064) (xy 129.7 68.1) (xy 135.9 74.3) (xy 135.824 120.2) (xy 162.204 120.2)
 				(xy 162.264 59.1) (xy 157.035 59.1) (xy 157.035 48.26) (xy 108.585 48.26)
 			)
